File: IRis.kicad_pcb (KiCad board)
At the start: 2 copper layers, 31.3 x 31.3 mm, 24 parts, among them P1 Power In, P2 Digital Out, Q1 MMBF4117, U1 TSV911ILT, U2 TLV3201

Commit message: Update to v1.3
Parts:
- removed LOGO: , LOGOS:WeatheredSecurityLogo
- removed P2: Digital Out, Pin_Headers:Pin_Header_Straight_1x02
- added BT1: 3v, CR2032:MPD BH32T-C, B.Cu at (142.2, 99.6)
- added Q2: MMBF4117, TO_SOT_Packages_SMD:SOT-23, F.Cu at (151.1, 96.3)
- added Q3: MMBF4117, TO_SOT_Packages_SMD:SOT-23, F.Cu at (151.1, 93.0)
- P1: value Power In -> Digital Out
- R10: value 10 -> 100
- moved P1 25.8 mm to (155.7, 100.8), turned to 180 degrees
- moved R6 16.0 mm to (134.1, 104.6), turned to 0 degrees
- moved C4 13.8 mm to (135.4, 100.6)
- moved R7 13.3 mm to (146.1, 110.0), turned to 0 degrees
- moved R4 13.2 mm to (146.8, 90.4), turned to 90 degrees
- moved C1 9.37 mm to (137.2, 93.2), turned to 270 degrees
- moved C2 8.89 mm to (144.0, 85.9), turned to 0 degrees
- moved R2 8.21 mm to (140.0, 87.6), turned to 0 degrees
- moved R3 7.38 mm to (140.0, 85.9), turned to 180 degrees
- moved C3 6.82 mm to (145.0, 90.4), turned to 270 degrees
- moved R1 6.59 mm to (139.2, 93.2), turned to 270 degrees
- moved R10 4.06 mm to (146.1, 108.0)
- moved R5 3.25 mm to (148.6, 91.4)
- moved Q1 2.34 mm to (147.8, 95.2)
- moved C7 0.80 mm to (132.8, 100.6)
Connections:
- P1 pad 1: +5V -> Net-(P1-Pad1)
- R10 pad 2: Net-(P2-Pad1) -> Net-(P1-Pad1)
- R5 pad 1: Net-(Q1-Pad3) -> Net-(Q3-Pad3)
Routing:
- net +5V: track 34.2 -> 8.58 mm, vias 0 -> 4
- net Net-(P2-Pad1): track 14.4 -> 0.00 mm, vias 1 -> 0
- net Net-(P1-Pad1): track 0.00 -> 13.9 mm
- net Net-(C5-Pad2): track 17.4 -> 3.74 mm, vias 2 -> 0
- net Net-(C3-Pad2): track 14.2 -> 3.96 mm
- net Net-(C1-Pad2): track 23.9 -> 15.8 mm, vias 1 -> 0
- net Net-(Q2-Pad3): track 0.00 -> 4.25 mm
- net Net-(R10-Pad1): track 5.86 -> 1.91 mm
- net Net-(C1-Pad1): track 19.6 -> 23.5 mm
- net Net-(C2-Pad1): track 9.42 -> 5.80 mm
- net Net-(C4-Pad1): track 13.8 -> 12.0 mm
- net Net-(Q3-Pad3): track 0.00 -> 1.72 mm
